File: Automotive Monitoring System CANBus Sensor/CANBus-MCP2551.kicad_sch (KiCad schematic)
At the start: 5 parts, among them J4 Conn_01x02, U3 MCP2551-I-SN

Commit message: ok updated the footprints. now toi get the DRC and a then PCB layout
Parts:
- D1: footprint SOT65P210X110-3N -> SamacSys_Parts:SOT65P210X110-3N
- J4: footprint (none) -> Connector_PinHeader_2.54mm:PinHeader_1x02_P2.54mm_Vertical
- R4, R6: footprint (none) -> Resistor_THT:R_Axial_DIN0207_L6.3mm_D2.5mm_P2.54mm_Vertical
Changed lines of the file:
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@@
 			)
 		)
-		(property "Footprint" "SOT65P210X110-3N"
+		(property "Footprint" "SamacSys_Parts:SOT65P210X110-3N"
 			(at 129.54 116.84 0)
 			(effects
@@
 			)
 		)
-		(property "Footprint" ""
+		(property "Footprint" "Connector_PinHeader_2.54mm:PinHeader_1x02_P2.54mm_Vertical"
 			(at 181.61 67.31 0)
 			(effects
@@
 			)
 		)
-		(property "Footprint" ""
+		(property "Footprint" "Resistor_THT:R_Axial_DIN0207_L6.3mm_D2.5mm_P2.54mm_Vertical"
 			(at 172.212 73.66 90)
 			(effects
@@
 			)
 		)
-		(property "Footprint" ""
+		(property "Footprint" "Resistor_THT:R_Axial_DIN0207_L6.3mm_D2.5mm_P2.54mm_Vertical"
 			(at 92.202 83.82 90)
 			(effects
