File: Automotive Monitoring System CANBus Sensor/BareMinAtmel328P.kicad_sch (KiCad schematic)
At the start: 8 parts, among them J1 ICSP, J2 TTL_Programmer, U1 ATmega328P-P, Y1 Crystal

Commit message: have the basic schems in need to assign footprints and do the PCB layout.
Parts:
- C1, C2: value C -> 22nf
- C3: value C -> 100nf
- R1: value R -> 10k
- Y1: value Crystal -> 16MHz
Changed lines of the file:
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@@
 			)
 		)
-		(property "Value" "C"
+		(property "Value" "22nf"
 			(at 208.28 64.77 90)
 			(effects
@@
 			)
 		)
-		(property "Value" "C"
+		(property "Value" "100nf"
 			(at 60.96 85.09 90)
 			(effects
@@
 			)
 		)
-		(property "Value" "Crystal"
+		(property "Value" "16MHz"
 			(at 199.39 77.4699 90)
 			(effects
@@
 			)
 		)
-		(property "Value" "R"
+		(property "Value" "10k"
 			(at 195.58 92.7099 0)
 			(effects
@@
 			)
 		)
-		(property "Value" "C"
+		(property "Value" "22nf"
 			(at 208.28 77.47 90)
 			(effects

Commit message: ok updated the footprints. now toi get the DRC and a then PCB layout
Parts:
- C1, C2, C3: footprint (none) -> Capacitor_SMD:C_1206_3216Metric_Pad1.33x1.80mm_HandSolder
- J1: footprint (none) -> Connector_PinHeader_2.54mm:PinHeader_2x03_P2.54mm_Vertical_SMD
- J2: footprint (none) -> Connector_PinHeader_2.54mm:PinHeader_1x06_P2.54mm_Vertical
- R1: footprint (none) -> Resistor_THT:R_Axial_DIN0207_L6.3mm_D2.5mm_P2.54mm_Vertical
- Y1: footprint (none) -> Crystal:Crystal_HC49-U_Vertical
Changed lines of the file:
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@@
 			)
 		)
-		(property "Footprint" ""
+		(property "Footprint" "Connector_PinHeader_2.54mm:PinHeader_2x03_P2.54mm_Vertical_SMD"
 			(at 43.18 49.53 0)
 			(effects
@@
 			)
 		)
-		(property "Footprint" ""
+		(property "Footprint" "Capacitor_SMD:C_1206_3216Metric_Pad1.33x1.80mm_HandSolder"
 			(at 212.09 68.8848 0)
 			(effects
@@
 			)
 		)
-		(property "Footprint" ""
+		(property "Footprint" "Connector_PinHeader_2.54mm:PinHeader_1x06_P2.54mm_Vertical"
 			(at 40.64 82.55 0)
 			(effects
@@
 			)
 		)
-		(property "Footprint" ""
+		(property "Footprint" "Capacitor_SMD:C_1206_3216Metric_Pad1.33x1.80mm_HandSolder"
 			(at 64.77 89.2048 0)
 			(effects
@@
 			)
 		)
-		(property "Footprint" ""
+		(property "Footprint" "Crystal:Crystal_HC49-U_Vertical"
 			(at 195.58 76.2 0)
 			(effects
@@
 			)
 		)
-		(property "Footprint" ""
+		(property "Footprint" "Resistor_THT:R_Axial_DIN0207_L6.3mm_D2.5mm_P2.54mm_Vertical"
 			(at 191.262 91.44 90)
 			(effects
@@
 			)
 		)
-		(property "Footprint" ""
+		(property "Footprint" "Capacitor_SMD:C_1206_3216Metric_Pad1.33x1.80mm_HandSolder"
 			(at 212.09 81.5848 0)
 			(effects

Commit message: tweaked footprints and made a bunch SMD for space saving. getting the board mostly placed before routing.
Parts:
- R1: footprint Resistor_THT:R_Axial_DIN0207_L6.3mm_D2.5mm_P2.54mm_Vertical -> Resistor_SMD:R_1206_3216Metric_Pad1.30x1.75mm_HandSolder
Changed lines of the file:
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@@
 			)
 		)
-		(property "Footprint" "Resistor_THT:R_Axial_DIN0207_L6.3mm_D2.5mm_P2.54mm_Vertical"
+		(property "Footprint" "Resistor_SMD:R_1206_3216Metric_Pad1.30x1.75mm_HandSolder"
 			(at 191.262 91.44 90)
 			(effects

Commit message: ammending my last commit to have the correct cap values of 22pF
Parts:
- C1, C2: value 22nf -> 22pf
Changed lines of the file:
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@@
 			)
 		)
-		(property "Value" "22nf"
+		(property "Value" "22pf"
 			(at 208.28 64.77 90)
 			(effects
@@
 			)
 		)
-		(property "Value" "22nf"
+		(property "Value" "22pf"
 			(at 208.28 77.47 90)
 			(effects
