File: AMS - CANBus Sensor - Pressure/BareMinAtmel328P.kicad_sch (KiCad schematic)
At the start: 8 parts, among them J1 ICSP, J2 TTL_Programmer, U1 ATmega328P-P, Y1 16MHz

Commit message: wip for this trying to figure out if i want to go completely SMD with this or not.
Parts:
- renumbered C3 to C1, C1 to C3, J2 to J3, J1 to J4, R1 to R4, U1 to U2
Changed lines of the file:
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@@
 		(dnp no)
 		(fields_autoplaced yes)
-		(property "Reference" "J1"
+		(property "Reference" "J4"
 			(at 44.45 40.64 0)
 			(effects
@@
 		)
 		(instances
-			(project "Automotive Monitoring System CANBus Sensor"
-				(path "/1c8b441e-37da-469b-a62d-a2093a833f7a/8782b0ef-1b0c-41b9-8665-2e7da5446ba9"
-					(reference "J1")
+			(project "AMS - CANBus Sensor - Pressure"
+				(path "/1c8b441e-37da-469b-a62d-a2093a833f7a/8782b0ef-1b0c-41b9-8665-2e7da5446ba9"
+					(reference "J4")
 					(unit 1)
 				)
@@
 		)
 		(instances
-			(project "Automotive Monitoring System CANBus Sensor"
+			(project "AMS - CANBus Sensor - Pressure"
 				(path "/1c8b441e-37da-469b-a62d-a2093a833f7a/8782b0ef-1b0c-41b9-8665-2e7da5446ba9"
 					(reference "C2")
@@
 		(on_board yes)
 		(dnp no)
-		(property "Reference" "J2"
+		(property "Reference" "J3"
 			(at 38.1 82.5499 0)
 			(effects
@@
 		)
 		(instances
-			(project "Automotive Monitoring System CANBus Sensor"
-				(path "/1c8b441e-37da-469b-a62d-a2093a833f7a/8782b0ef-1b0c-41b9-8665-2e7da5446ba9"
-					(reference "J2")
+			(project "AMS - CANBus Sensor - Pressure"
+				(path "/1c8b441e-37da-469b-a62d-a2093a833f7a/8782b0ef-1b0c-41b9-8665-2e7da5446ba9"
+					(reference "J3")
 					(unit 1)
 				)
@@
 		(dnp no)
 		(fields_autoplaced yes)
-		(property "Reference" "C3"
+		(property "Reference" "C1"
 			(at 60.96 82.55 90)
 			(effects
@@
 		)
 		(instances
-			(project "Automotive Monitoring System CANBus Sensor"
-				(path "/1c8b441e-37da-469b-a62d-a2093a833f7a/8782b0ef-1b0c-41b9-8665-2e7da5446ba9"
-					(reference "C3")
+			(project "AMS - CANBus Sensor - Pressure"
+				(path "/1c8b441e-37da-469b-a62d-a2093a833f7a/8782b0ef-1b0c-41b9-8665-2e7da5446ba9"
+					(reference "C1")
 					(unit 1)
 				)
@@
 		)
 		(instances
-			(project "Automotive Monitoring System CANBus Sensor"
+			(project "AMS - CANBus Sensor - Pressure"
 				(path "/1c8b441e-37da-469b-a62d-a2093a833f7a/8782b0ef-1b0c-41b9-8665-2e7da5446ba9"
 					(reference "Y1")
@@
 		(dnp no)
 		(fields_autoplaced yes)
-		(property "Reference" "R1"
+		(property "Reference" "R4"
 			(at 195.58 90.1699 0)
 			(effects
@@
 		)
 		(instances
-			(project "Automotive Monitoring System CANBus Sensor"
-				(path "/1c8b441e-37da-469b-a62d-a2093a833f7a/8782b0ef-1b0c-41b9-8665-2e7da5446ba9"
-					(reference "R1")
+			(project "AMS - CANBus Sensor - Pressure"
+				(path "/1c8b441e-37da-469b-a62d-a2093a833f7a/8782b0ef-1b0c-41b9-8665-2e7da5446ba9"
+					(reference "R4")
 					(unit 1)
 				)
@@
 		(dnp no)
 		(fields_autoplaced yes)
-		(property "Reference" "C1"
+		(property "Reference" "C3"
 			(at 208.28 74.93 90)
 			(effects
@@
 		)
 		(instances
-			(project "Automotive Monitoring System CANBus Sensor"
-				(path "/1c8b441e-37da-469b-a62d-a2093a833f7a/8782b0ef-1b0c-41b9-8665-2e7da5446ba9"
-					(reference "C1")
+			(project "AMS - CANBus Sensor - Pressure"
+				(path "/1c8b441e-37da-469b-a62d-a2093a833f7a/8782b0ef-1b0c-41b9-8665-2e7da5446ba9"
+					(reference "C3")
 					(unit 1)
 				)
@@
 		(dnp no)
 		(fields_autoplaced yes)
-		(property "Reference" "U1"
+		(property "Reference" "U2"
 			(at 118.11 52.1014 0)
 			(effects
@@
 		)
 		(instances
-			(project "Automotive Monitoring System CANBus Sensor"
-				(path "/1c8b441e-37da-469b-a62d-a2093a833f7a/8782b0ef-1b0c-41b9-8665-2e7da5446ba9"
-					(reference "U1")
-					(unit 1)
-				)
+			(project "AMS - CANBus Sensor - Pressure"
+				(path "/1c8b441e-37da-469b-a62d-a2093a833f7a/8782b0ef-1b0c-41b9-8665-2e7da5446ba9"
+					(reference "U2")
+					(unit 1)
+				)
