File: AMS - CANBus Sensor - Pressure/CANBUS-MCP2515.kicad_sch (KiCad schematic)
At the start: 7 parts, among them U4 MCP2515-xSO, Y2 16MHz

Commit message: wip for this trying to figure out if i want to go completely SMD with this or not.
Parts:
- renumbered C6 to C4, C7 to C5, C5 to C6, C4 to C7, U4 to U3
Changed lines of the file:
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@@
 		(dnp no)
 		(fields_autoplaced yes)
-		(property "Reference" "U4"
+		(property "Reference" "U3"
 			(at 138.0841 55.88 0)
 			(effects
@@
 		)
 		(instances
-			(project "Automotive Monitoring System CANBus Sensor"
-				(path "/1c8b441e-37da-469b-a62d-a2093a833f7a/7d96c4e1-93d6-45eb-8bfa-0469ecf38441"
-					(reference "U4")
+			(project "AMS - CANBus Sensor - Pressure"
+				(path "/1c8b441e-37da-469b-a62d-a2093a833f7a/7d96c4e1-93d6-45eb-8bfa-0469ecf38441"
+					(reference "U3")
 					(unit 1)
 				)
@@
 		(dnp no)
 		(fields_autoplaced yes)
-		(property "Reference" "C5"
+		(property "Reference" "C6"
 			(at 104.14 40.64 90)
 			(effects
@@
 		)
 		(instances
-			(project "Automotive Monitoring System CANBus Sensor"
-				(path "/1c8b441e-37da-469b-a62d-a2093a833f7a/7d96c4e1-93d6-45eb-8bfa-0469ecf38441"
-					(reference "C5")
+			(project "AMS - CANBus Sensor - Pressure"
+				(path "/1c8b441e-37da-469b-a62d-a2093a833f7a/7d96c4e1-93d6-45eb-8bfa-0469ecf38441"
+					(reference "C6")
 					(unit 1)
 				)
@@
 		)
 		(instances
-			(project "Automotive Monitoring System CANBus Sensor"
+			(project "AMS - CANBus Sensor - Pressure"
 				(path "/1c8b441e-37da-469b-a62d-a2093a833f7a/7d96c4e1-93d6-45eb-8bfa-0469ecf38441"
 					(reference "R5")
@@
 		)
 		(instances
-			(project "Automotive Monitoring System CANBus Sensor"
+			(project "AMS - CANBus Sensor - Pressure"
 				(path "/1c8b441e-37da-469b-a62d-a2093a833f7a/7d96c4e1-93d6-45eb-8bfa-0469ecf38441"
 					(reference "Y2")
@@
 		(dnp no)
 		(fields_autoplaced yes)
-		(property "Reference" "C6"
+		(property "Reference" "C4"
 			(at 68.58 76.2 90)
 			(effects
@@
 		)
 		(instances
-			(project "Automotive Monitoring System CANBus Sensor"
-				(path "/1c8b441e-37da-469b-a62d-a2093a833f7a/7d96c4e1-93d6-45eb-8bfa-0469ecf38441"
-					(reference "C6")
+			(project "AMS - CANBus Sensor - Pressure"
+				(path "/1c8b441e-37da-469b-a62d-a2093a833f7a/7d96c4e1-93d6-45eb-8bfa-0469ecf38441"
+					(reference "C4")
 					(unit 1)
 				)
@@
 		(dnp no)
 		(fields_autoplaced yes)
-		(property "Reference" "C4"
+		(property "Reference" "C7"
 			(at 116.84 40.64 90)
 			(effects
@@
 		)
 		(instances
-			(project "Automotive Monitoring System CANBus Sensor"
-				(path "/1c8b441e-37da-469b-a62d-a2093a833f7a/7d96c4e1-93d6-45eb-8bfa-0469ecf38441"
-					(reference "C4")
+			(project "AMS - CANBus Sensor - Pressure"
+				(path "/1c8b441e-37da-469b-a62d-a2093a833f7a/7d96c4e1-93d6-45eb-8bfa-0469ecf38441"
+					(reference "C7")
 					(unit 1)
 				)
@@
 		(dnp no)
 		(fields_autoplaced yes)
-		(property "Reference" "C7"
+		(property "Reference" "C5"
 			(at 68.58 88.9 90)
 			(effects
@@
 		)
 		(instances
-			(project "Automotive Monitoring System CANBus Sensor"
-				(path "/1c8b441e-37da-469b-a62d-a2093a833f7a/7d96c4e1-93d6-45eb-8bfa-0469ecf38441"
-					(reference "C7")
-					(unit 1)
-				)
+			(project "AMS - CANBus Sensor - Pressure"
+				(path "/1c8b441e-37da-469b-a62d-a2093a833f7a/7d96c4e1-93d6-45eb-8bfa-0469ecf38441"
+					(reference "C5")
+					(unit 1)
+				)
