File: AMS - CANBus Sensor - Pressure/CANBus-MCP2551.kicad_sch (KiCad schematic)
At the start: 5 parts, among them J4 Conn_01x02, U3 MCP2551-I-SN

Commit message: wip for this trying to figure out if i want to go completely SMD with this or not.
Parts:
- renumbered J4 to J5, R4 to R6, R6 to R7, U3 to U4
Changed lines of the file:
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@@
 		)
 		(instances
-			(project "Automotive Monitoring System CANBus Sensor"
+			(project "AMS - CANBus Sensor - Pressure"
 				(path "/1c8b441e-37da-469b-a62d-a2093a833f7a/5df34325-0121-481e-982d-7498a0311385"
 					(reference "D1")
@@
 		(dnp no)
 		(fields_autoplaced yes)
-		(property "Reference" "J4"
+		(property "Reference" "J5"
 			(at 184.15 67.3099 0)
 			(effects
@@
 		)
 		(instances
-			(project "Automotive Monitoring System CANBus Sensor"
-				(path "/1c8b441e-37da-469b-a62d-a2093a833f7a/5df34325-0121-481e-982d-7498a0311385"
-					(reference "J4")
+			(project "AMS - CANBus Sensor - Pressure"
+				(path "/1c8b441e-37da-469b-a62d-a2093a833f7a/5df34325-0121-481e-982d-7498a0311385"
+					(reference "J5")
 					(unit 1)
 				)
@@
 		(dnp no)
 		(fields_autoplaced yes)
-		(property "Reference" "U3"
+		(property "Reference" "U4"
 			(at 112.6841 62.23 0)
 			(effects
@@
 		)
 		(instances
-			(project "Automotive Monitoring System CANBus Sensor"
-				(path "/1c8b441e-37da-469b-a62d-a2093a833f7a/5df34325-0121-481e-982d-7498a0311385"
-					(reference "U3")
+			(project "AMS - CANBus Sensor - Pressure"
+				(path "/1c8b441e-37da-469b-a62d-a2093a833f7a/5df34325-0121-481e-982d-7498a0311385"
+					(reference "U4")
 					(unit 1)
 				)
@@
 		(dnp no)
 		(fields_autoplaced yes)
-		(property "Reference" "R6"
+		(property "Reference" "R7"
 			(at 176.53 72.3899 0)
 			(effects
@@
 		)
 		(instances
-			(project "Automotive Monitoring System CANBus Sensor"
-				(path "/1c8b441e-37da-469b-a62d-a2093a833f7a/5df34325-0121-481e-982d-7498a0311385"
-					(reference "R6")
+			(project "AMS - CANBus Sensor - Pressure"
+				(path "/1c8b441e-37da-469b-a62d-a2093a833f7a/5df34325-0121-481e-982d-7498a0311385"
+					(reference "R7")
 					(unit 1)
 				)
@@
 		(dnp no)
 		(fields_autoplaced yes)
-		(property "Reference" "R4"
+		(property "Reference" "R6"
 			(at 96.52 82.5499 0)
 			(effects
@@
 		)
 		(instances
-			(project "Automotive Monitoring System CANBus Sensor"
-				(path "/1c8b441e-37da-469b-a62d-a2093a833f7a/5df34325-0121-481e-982d-7498a0311385"
-					(reference "R4")
-					(unit 1)
-				)
+			(project "AMS - CANBus Sensor - Pressure"
+				(path "/1c8b441e-37da-469b-a62d-a2093a833f7a/5df34325-0121-481e-982d-7498a0311385"
+					(reference "R6")
+					(unit 1)
+				)

Commit message: ready for fab
Parts:
- D1: footprint SamacSys_Parts:SOT65P210X110-3N -> SOT65P210X110-3N
Changed lines of the file:
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@@
 			)
 		)
-		(property "Footprint" "SamacSys_Parts:SOT65P210X110-3N"
+		(property "Footprint" "SOT65P210X110-3N"
 			(at 129.54 116.84 0)
 			(effects
