File: AMS - CANBus Sensor - Pressure/BufferedADC.kicad_sch (KiCad schematic)
At the start: 9 parts, among them IC1 OPA4340UA

Commit message: ready for fab
Parts:
- removed IC1: OPA4340UA, SamacSys_Parts:SOIC127P600X175-14N, symbol Samac_Sys:OPA4340UA
- added IC2: OPA4340UA, SOIC127P600X175-14N, symbol SamacSys_Parts:OPA4340UA
Connections:
- net ADCIN1: now also IC2.3 (+IN_A)
- net ADCIN2: now also IC2.5 (+IN_B)
- net ADCIN3: now also IC2.10 (+IN_C)
- net ADCIN4: now also IC2.12 (+IN_D)
- net ADCOUT1: now also IC2.1 (OUT_A), IC2.2 (-IN_A)
- net ADCOUT2: now also IC2.6 (-IN_B), IC2.7 (OUT_B)
- net ADCOUT3: now also IC2.8 (OUT_C), IC2.9 (-IN_C)
- net ADCOUT4: now also IC2.13 (-IN_D), IC2.14 (OUT_D)
- net GND: now also IC2.11 (V-)
- net Vin: now also IC2.4 (V+)
Other:
- moved on the sheet: R11

Commit message: removed un-needed BufferedADC.kicad_sch from IO and Temp boards as that was copied over.
R8,9,14,15 100k resistors were removed from the ADC input and in parallel witht he 200k pots and then moved to be in series with the pots and changed to 1k
Parts:
- removed R14, R15, R8, R9: 100K, Resistor_SMD:R_1206_3216Metric_Pad1.30x1.75mm_HandSolder, symbol Device:R
