File: Automotive Monitoring System CANBus Sensor SMD Processor/Automotive Monitoring System CANBus Sensor SMD Processor.kicad_sch (KiCad schematic)
At the start: 10 parts, among them J3 Conn_02x10_Odd_Even, J5 Power_And_CAN, Q1 IRF9Z34NPBF, U2 178.6165.0001

Commit message: wip for RPM
Parts:
- removed U2: 178.6165.0001, SamacSys_Parts:17861650001, symbol SamacSys_Parts:178.6165.0001
- added U1: 3568, 3568, symbol SamacSys_Parts:3568
Connections:
- net +VDC: now also U1.3, U1.4
- net at Q1.3: now also U1.1, U1.2
