File: AMS - CANBus Sensor - Temperature - RTD/MAX31865AAP+.kicad_sch (KiCad schematic)
At the start: 8 parts, among them IC1 MAX31865AAP+, J2 Conn_01x02, J6 Conn_01x03, J7 Conn_01x02

Commit message: RTD Sensor V1.1 Rev B
swapped 0.1 MM pitch header pins for 0.1In pitch
Parts:
- J2, J7: footprint Connector_PinHeader_1.00mm:PinHeader_1x02_P1.00mm_Vertical_SMD_Pin1Left -> Connector_PinHeader_2.54mm:PinHeader_1x02_P2.54mm_Vertical_SMD_Pin1Right
- J6: footprint Connector_PinHeader_1.00mm:PinHeader_1x03_P1.00mm_Vertical_SMD_Pin1Left -> Connector_PinHeader_2.54mm:PinHeader_1x03_P2.54mm_Vertical_SMD_Pin1Right
Changed lines of the file:
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@@
 		)
 		(instances
-			(project "AMS - CANBus Sensor - Temperature"
+			(project "AMS - CANBus Sensor - Temperature - RTD"
 				(path "/1c8b441e-37da-469b-a62d-a2093a833f7a/2e0562a2-0f62-4c3a-a7f1-916335767d69"
 					(reference "IC1")
@@
 		)
 		(instances
-			(project "AMS - CANBus Sensor - Temperature"
+			(project "AMS - CANBus Sensor - Temperature - RTD"
 				(path "/1c8b441e-37da-469b-a62d-a2093a833f7a/2e0562a2-0f62-4c3a-a7f1-916335767d69"
 					(reference "C9")
@@
 		)
 		(instances
-			(project "AMS - CANBus Sensor - Temperature"
+			(project "AMS - CANBus Sensor - Temperature - RTD"
 				(path "/1c8b441e-37da-469b-a62d-a2093a833f7a/2e0562a2-0f62-4c3a-a7f1-916335767d69"
 					(reference "C8")
@@
 		)
 		(instances
-			(project "AMS - CANBus Sensor - Temperature"
+			(project "AMS - CANBus Sensor - Temperature - RTD"
 				(path "/1c8b441e-37da-469b-a62d-a2093a833f7a/2e0562a2-0f62-4c3a-a7f1-916335767d69"
 					(reference "R8")
@@
 			)
 		)
-		(property "Footprint" "Connector_PinHeader_1.00mm:PinHeader_1x02_P1.00mm_Vertical_SMD_Pin1Left"
+		(property "Footprint" "Connector_PinHeader_2.54mm:PinHeader_1x02_P2.54mm_Vertical_SMD_Pin1Right"
 			(at 97.79 95.25 0)
 			(effects
@@
 		)
 		(instances
-			(project "AMS - CANBus Sensor - Temperature"
+			(project "AMS - CANBus Sensor - Temperature - RTD"
 				(path "/1c8b441e-37da-469b-a62d-a2093a833f7a/2e0562a2-0f62-4c3a-a7f1-916335767d69"
 					(reference "J2")
@@
 			)
 		)
-		(property "Footprint" "Connector_PinHeader_1.00mm:PinHeader_1x03_P1.00mm_Vertical_SMD_Pin1Left"
+		(property "Footprint" "Connector_PinHeader_2.54mm:PinHeader_1x03_P2.54mm_Vertical_SMD_Pin1Right"
 			(at 97.79 109.22 0)
 			(effects
@@
 		)
 		(instances
-			(project "AMS - CANBus Sensor - Temperature"
+			(project "AMS - CANBus Sensor - Temperature - RTD"
 				(path "/1c8b441e-37da-469b-a62d-a2093a833f7a/2e0562a2-0f62-4c3a-a7f1-916335767d69"
 					(reference "J6")
@@
 			)
 		)
-		(property "Footprint" "Connector_PinHeader_1.00mm:PinHeader_1x02_P1.00mm_Vertical_SMD_Pin1Left"
+		(property "Footprint" "Connector_PinHeader_2.54mm:PinHeader_1x02_P2.54mm_Vertical_SMD_Pin1Right"
 			(at 191.77 97.79 0)
 			(effects
@@
 		)
 		(instances
-			(project "AMS - CANBus Sensor - Temperature"
+			(project "AMS - CANBus Sensor - Temperature - RTD"
 				(path "/1c8b441e-37da-469b-a62d-a2093a833f7a/2e0562a2-0f62-4c3a-a7f1-916335767d69"
 					(reference "J7")
@@
 		)
 		(instances
-			(project "AMS - CANBus Sensor - Temperature"
+			(project "AMS - CANBus Sensor - Temperature - RTD"
 				(path "/1c8b441e-37da-469b-a62d-a2093a833f7a/2e0562a2-0f62-4c3a-a7f1-916335767d69"
 					(reference "C10")
