File: AMS - CANBus - Dinger/AMS - CANBus - Dinger.kicad_sch (KiCad schematic)
At the start: 17 parts, among them J1 TTL_Programmer, J3 Power_And_CAN, Q1 IRF9Z34NPBF, U1 178.6165.0001, U2 ATmega328-P, Y1 Crystal

Commit message: initial placement of parts
Parts:
- added U8: 178.6165.0001, SamacSys_Parts:17861650001, symbol SamacSys_Parts:178.6165.0001
Connections:
- net at Q1.3, U1.3, U1.4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: now also U8.3, U8.4, U8.5, U8.6
- new net +VSW: U8.1, U8.2, U8.7, U8.8
Other:
- sheet Output ports: added OutputVS; removed none
- sheet Output1 ports: added OutputVS; removed none
- sheet Output2 ports: added OutputVS; removed none
- moved on the sheet: Powerboard1
