File: AMS - CANBus - Dinger/AMS - CANBus - Dinger.kicad_pcb (KiCad board)
At the start: 2 copper layers, 71.1 x 111 mm, 75 parts, among them J1 TTL_Programmer, J2 Conn_01x02, P1 Screw_Terminal_01x02, P2 Screw_Terminal_01x02, Q1 IRF9Z34NPBF, Q10 IRF9Z34NPBF, Q2 2N7000, Q3 2N7000, Q4 IRF9Z34NPBF, Q5 2N7000, Q6 2N7000, Q7 2N7000, Q8 IRF9Z34NPBF, Q9 2N7000, U1 178.6165.0001, U2 ATmega328-P, U3 LTV-817, U4 LTV-817, U5 LTV-817, U6 MCP2515-xSO, U7 MCP2551-I-SN, Y1 Crystal, Y2 16MHz

Commit message: initial placement of parts
Parts:
- removed P1, P2: Screw_Terminal_01x02, TerminalBlock_Phoenix:TerminalBlock_Phoenix_MKDS-1,5-2-5.08_1x02_P5.08mm_Horizontal
- added J3: Power_And_CAN, TerminalBlock_Phoenix:TerminalBlock_Phoenix_MPT-0,5-4-2.54_1x04_P2.54mm_Horizontal, F.Cu at (131.6, 66.2)
- added U8: 178.6165.0001, SamacSys_Parts:17861650001, F.Cu at (105.7, 61.5)
- C10, C14, C2, C8, C9, D9, R1, R10, R11, R12, R13, R14, R15, R16, R17, R18, R19, R2, R20, R21, R22, R23, R24, R25, R5, R6, R7, R8, R9, U6, U7: moved to B.Cu
- R27, R28: footprint Resistor_SMD:R_1206_3216Metric_Pad1.30x1.75mm_HandSolder -> Resistor_THT:R_Axial_DIN0204_L3.6mm_D1.6mm_P1.90mm_Vertical
- moved C10 264.2 mm to (82.3, 98.2)
- moved C12 239.3 mm to (86.8, 48.7)
- moved C11 239.1 mm to (86.6, 63.3), turned to 180 degrees
- moved Y2 239.1 mm to (86.7, 53.6), turned to -90 degrees
- moved Y1 235.4 mm to (122.8, 99.5), turned to 90 degrees
- moved U6 231.2 mm to (104.4, 50.1)
- moved R26 211.8 mm to (114.6, 53.5), turned to 180 degrees
- moved C14 211.8 mm to (114.6, 51.1)
- moved C13 211.6 mm to (114.6, 51.0)
- moved R28 202.6 mm to (122.6, 70.9)
- moved U7 200.9 mm to (132.3, 75.2)
- moved U5 195.0 mm to (78.4, 90.9), turned to 0 degrees
- moved D9 193.3 mm to (138.3, 73.0), turned to -90 degrees
- moved R27 190.0 mm to (134.8, 79.1)
- moved R16 186.5 mm to (82.2, 95.8)
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Connections:
- net /CANBUS-MCP2551/CANH renamed CANBUS_H
- net /CANBUS-MCP2551/CANL renamed CANBUS_L
- Q10 pad 3: +VDC -> +VSW
- Q4 pad 3: +VDC -> +VSW
- Q8 pad 3: +VDC -> +VSW
- R10 pad 1: +VDC -> +VSW
- R21 pad 1: +VDC -> +VSW
- R24 pad 1: +VDC -> +VSW
- Z3 pad 1: +VDC -> +VSW
- Z4 pad 1: +VDC -> +VSW
- Z5 pad 1: +VDC -> +VSW
Routing:
- net Net-(Q1-Pad3): track 0.00 -> 51.8 mm
- net +VSW: track 0.00 -> 12.0 mm
- net +VDC: track 0.00 -> 12.0 mm
- net Net-(J3-Pin_1): track 0.00 -> 7.34 mm
Other:
- board text added: "1 amp"
- board text added: "120 Ohm CAN Bus Resistor"
- board text added: "12V"
- board text added: "3 amp"
- board text added: "AMS - Dinger V1.0.0"
- board text added: "CH"
- board text added: "CL"
- board text added: "GND"
- board text removed: "+"
- board text removed: "-"
- board text removed: "2amp"
- board text removed: "Basic Bitch 328p Thingy V2.0.0"
- board text removed: "ISCP"
- board text removed: "RX"
- board text removed: "TTL"
- board text removed: "TX"

Commit message: pre freerouting
Parts:
- moved R2 1.78 mm to (120.7, 132.8)
- moved C2 1.06 mm to (119.2, 121.3)
Routing:
- net GND: track 0.00 -> 296.0 mm, vias 0 -> 1
- net +VSW: track 12.0 -> 167.5 mm, vias 0 -> 3
- net +5V: track 0.00 -> 102.7 mm, vias 0 -> 7
- net /Input1/Input: track 0.00 -> 35.3 mm
- net /Output2/Output: track 0.00 -> 31.7 mm
- net /Input2/Input: track 0.00 -> 27.9 mm
- net /Output1/Output: track 0.00 -> 27.4 mm
- net /Output/Output: track 0.00 -> 27.1 mm
- net CANBUS_L: track 0.00 -> 27.1 mm
- net /Input/Input: track 0.00 -> 25.4 mm
- net Net-(U6-OSC2): track 0.00 -> 23.1 mm, vias 0 -> 1
- net +VDC: track 12.0 -> 34.6 mm
- net Net-(U6-OSC1): track 0.00 -> 21.5 mm, vias 0 -> 1
- net Net-(Q8-Pad1): track 0.00 -> 21.2 mm
- net Net-(Q10-Pad1): track 0.00 -> 21.1 mm
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
Commit message: Dinger V1.0.0 Files done and submitted for FAB
Routing:
- net GND: track 296.0 -> 441.7 mm, vias 1 -> 2
- net +5V: track 102.7 -> 219.1 mm, vias 7 -> 9
- net Output2: track 4.70 -> 97.3 mm
- net MISO: track 0.00 -> 86.0 mm, vias 0 -> 2
- net Output3: track 4.13 -> 77.0 mm
- net SCK: track 0.00 -> 71.7 mm, vias 0 -> 4
- net D10: track 0.00 -> 70.2 mm, vias 0 -> 6
- net Input1: track 3.13 -> 72.0 mm, vias 0 -> 1
- net Output1: track 5.02 -> 70.6 mm, vias 0 -> 1
- net MOSI: track 0.00 -> 62.4 mm, vias 0 -> 2
- net D8: track 1.19 -> 63.4 mm, vias 0 -> 2
- net Input3: track 3.90 -> 64.0 mm, vias 0 -> 2
- net Input2: track 3.77 -> 53.4 mm, vias 0 -> 2
- net /CANBUS-MCP2515/TXtoCANTC: track 0.00 -> 46.7 mm, vias 0 -> 2
- net /CANBUS-MCP2515/RXtoCANTC: track 0.00 -> 45.0 mm, vias 0 -> 2
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