File: AMS - CANBus Sensor - Voltage/AMS - CANBus Sensor - Voltage.kicad_pcb (KiCad board)
At the start: 2 copper layers, 72.9 x 71.1 mm, 45 parts, among them IC2 OPA4340UA, J1 Power_And_CAN, J2 Power_And_CAN, J3 TTL_Programmer, J4 ICSP, J5 Conn_01x02, J6 Screw_Terminal_01x02, Q1 IRF9Z34NPBF, U1 3568, U2 ATmega328P-P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

Commit message: wip for this.
Parts:
- removed NTC1: 10k, Resistor_THT:R_Axial_DIN0207_L6.3mm_D2.5mm_P2.54mm_Vertical
- removed R3: 10k, Resistor_SMD:R_1206_3216Metric_Pad1.30x1.75mm_HandSolder
- added J7: Conn_01x02, Connector_PinHeader_2.54mm:PinHeader_1x02_P2.54mm_Vertical, F.Cu at (135.0, 92.6)
Connections:
- R12 pad 2: /BareMinAtmel328P/PC4-A4-SDA -> /BareMinAtmel328P/PC0-A0
- U2 pad 27: /BareMinAtmel328P/PC4-A4-SDA -> SDA
- U2 pad 28: /BareMinAtmel328P/PC5-A5-SCL -> SCL
Routing:
- net /BareMinAtmel328P/PC4-A4-SDA: track 62.3 -> 1.27 mm, vias 2 -> 0
- net /BareMinAtmel328P/PC0-A0: track 15.9 -> 0.00 mm
- net +5V: track 185.0 -> 175.2 mm
- net /BareMinAtmel328P/PC1-A1: track 53.8 -> 54.5 mm

Commit message: i think this is ready
Parts:
- D1: footprint SamacSys_Parts:SOT65P210X110-3N -> SamacSys:SOT65P210X110-3N
- IC2: footprint SamacSys_Parts:SOIC127P600X175-14N -> SamacSys:SOIC127P600X175-14N
- Q1: footprint SamacSys_Parts:TO254P469X1042X1967-3P -> SamacSys:TO254P469X1042X1967-3P
- Reset1: footprint SamacSys_Parts:TS0266160BK260LCRD -> SamacSys:TS0266160BK260LCRD
- U1, U5: footprint SamacSys_Parts:3568 -> SamacSys:3568
Connections:
- IC2 pad 13: /BareMinAtmel328P/PC4-A4-SDA -> /BareMinAtmel328P/PC0-A0
- IC2 pad 14: /BareMinAtmel328P/PC4-A4-SDA -> /BareMinAtmel328P/PC0-A0
Routing:
- net /BareMinAtmel328P/PC0-A0: track 0.00 -> 68.8 mm, vias 0 -> 3
- net /BufferedADC/ADCIN4: track 76.4 -> 45.2 mm, vias 1 -> 3
- net +5V: track 175.2 -> 202.3 mm, vias 1 -> 3
- net /BareMinAtmel328P/PB1-D9: track 108.6 -> 89.7 mm, vias 0 -> 3
- net SCL: track 0.00 -> 17.7 mm
- net SDA: track 0.00 -> 17.1 mm
- net /BufferedADC/ADCIN2: track 31.8 -> 46.9 mm, vias 1 -> 2
- net /BareMinAtmel328P/PB3-D11-MOSI: track 94.3 -> 79.3 mm, vias 1 -> 2
- net Net-(U3-~{RESET}): track 25.9 -> 39.6 mm
- net +VDC: track 40.0 -> 29.5 mm, vias 1 -> 0
- net CANBUS_L: track 35.8 -> 45.3 mm, vias 0 -> 1
- net GND: track 233.8 -> 224.3 mm, vias 6 -> 4
- net /BareMinAtmel328P/RESET: track 84.6 -> 76.9 mm, vias 2 -> 3
- net /BareMinAtmel328P/PC3-A3: track 72.6 -> 67.7 mm
- net Net-(J2-Pin_4): track 18.7 -> 23.6 mm, vias 0 -> 1
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Other:
- board text added: "AMS CANBus Voltage V2.0 Rev A"
- board text added: "SCL"
- board text added: "SDA"
- board text removed: "AMS CANBus Voltage V1.1 Rev A"
